File: cabsim/cabsim.kicad_sch (KiCad schematic)
At the start: 45 parts, among them J1 NJ3FD-V, J3 Conn_01x01, J4 Conn_01x01, J5 NJ3FD-V, U3 Op_Amp_Dual, U4 Opamp_Quad

Commit message: update pcb
Parts:
- C4: value 1n -> 3.3n
- C7: value 2.2n -> 3.3n
- R19: value 390 -> 330
- R5, R9: value 3.9k -> 3.3k
Other:
- moved on the sheet: C1, C10, C11, C12, C13, C14, C15, C16, C17, C2, C3, C4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

Commit message: update pcb and gitignore
Connections:
- net at C7.1, R15.1, R9.2: now also U4.1; no longer U4.14
- net at C7.2, R9.1, RV1.1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: now also U4.2 (-); no longer U4.13 (-)
- net at C4.1, C5.2, R6.2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: now also U4.14; no longer U4.1
- net at C4.2, R5.2, R6.1: now also U4.13 (-); no longer U4.2 (-)
- net at C2.1, R1.1: now also U4.12 (+); no longer U4.3 (+)
- net at C5.1, R8.2: now also U4.3 (+); no longer U4.12 (+)
Other:
- moved on the sheet: U4A, U4D
Changed lines of the file:
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@@
 	(symbol
 		(lib_id "Device:Opamp_Quad")
-		(at 97.79 36.83 0)
+		(at 148.59 39.37 0)
 		(unit 1)
 		(exclude_from_sim no)
@@
 		(fields_autoplaced yes)
 		(property "Reference" "U4"
-			(at 97.79 26.67 0)
+			(at 148.59 29.21 0)
 			(effects
 				(font
@@
 		)
 		(property "Value" "Opamp_Quad"
-			(at 97.79 29.21 0)
+			(at 148.59 31.75 0)
 			(effects
 				(font
@@
 		)
 		(property "Footprint" "1_trevortjes_lib:DIP-14"
-			(at 97.79 36.83 0)
+			(at 148.59 39.37 0)
 			(effects
 				(font
@@
 		)
 		(property "Datasheet" "~"
-			(at 97.79 36.83 0)
+			(at 148.59 39.37 0)
 			(effects
 				(font
@@
 		)
 		(property "Description" "Quad operational amplifier"
-			(at 97.79 36.83 0)
+			(at 148.59 39.37 0)
 			(effects
 				(font
@@
 		)
 		(property "Sim.Library" "${KICAD9_SYMBOL_DIR}/Simulation_SPICE.sp"
-			(at 97.79 36.83 0)
+			(at 148.59 39.37 0)
 			(effects
 				(font
@@
 		)
 		(property "Sim.Name" "kicad_builtin_opamp_quad"
-			(at 97.79 36.83 0)
+			(at 148.59 39.37 0)
 			(effects
 				(font
@@
 		)
 		(property "Sim.Device" "SUBCKT"
-			(at 97.79 36.83 0)
+			(at 148.59 39.37 0)
 			(effects
 				(font
@@
 		)
 		(property "Sim.Pins" "1=out1 2=in1- 3=in1+ 4=vcc 5=in2+ 6=in2- 7=out2 8=out3 9=in3- 10=in3+ 11=vee 12=in4+ 13=in4- 14=out4"
-			(at 97.79 36.83 0)
+			(at 148.59 39.37 0)
 			(effects
 				(font
@@
 	(symbol
 		(lib_id "Device:Opamp_Quad")
-		(at 148.59 39.37 0)
+		(at 97.79 36.83 0)
 		(unit 4)
 		(exclude_from_sim no)
@@
 		(fields_autoplaced yes)
 		(property "Reference" "U4"
-			(at 148.59 29.21 0)
+			(at 97.79 26.67 0)
 			(effects
 				(font
@@
 		)
 		(property "Value" "Opamp_Quad"
-			(at 148.59 31.75 0)
+			(at 97.79 29.21 0)
 			(effects
 				(font
@@
 		)
 		(property "Footprint" "1_trevortjes_lib:DIP-14"
-			(at 148.59 39.37 0)
+			(at 97.79 36.83 0)
 			(effects
 				(font
@@
 		)
 		(property "Datasheet" "~"
-			(at 148.59 39.37 0)
+			(at 97.79 36.83 0)
 			(effects
 				(font
@@
 		)
 		(property "Description" "Quad operational amplifier"
-			(at 148.59 39.37 0)
+			(at 97.79 36.83 0)
 			(effects
 				(font
@@
 		)
 		(property "Sim.Library" "${KICAD9_SYMBOL_DIR}/Simulation_SPICE.sp"
-			(at 148.59 39.37 0)
+			(at 97.79 36.83 0)
 			(effects
 				(font
@@
 		)
 		(property "Sim.Name" "kicad_builtin_opamp_quad"
-			(at 148.59 39.37 0)
+			(at 97.79 36.83 0)
 			(effects
 				(font
@@
 		)
 		(property "Sim.Device" "SUBCKT"
-			(at 148.59 39.37 0)
+			(at 97.79 36.83 0)
 			(effects
 				(font
@@
 		)
 		(property "Sim.Pins" "1=out1 2=in1- 3=in1+ 4=vcc 5=in2+ 6=in2- 7=out2 8=out3 9=in3- 10=in3+ 11=vee 12=in4+ 13=in4- 14=out4"
-			(at 148.59 39.37 0)
-			(effects
-				(font
+			(at 97.79 36.83 0)
+			(effects
+				(font
